Commit message: set joint 1 limit to full range

File: widowx_arm_description/urdf/widowx.urdf.xacro (robot description, xacro)
@@ -204,5 +204,5 @@
          <child link="${prefix}shoulder_link" />
          <axis xyz="0 0 1" />
-         <limit lower="-2.617" upper="2.617" effort="6" velocity="0.785" />
+	 <limit lower="-${M_PI}" upper="${M_PI}" effort="6" velocity="0.785" />
       </joint>
       <joint name="${prefix}joint_2" type="revolute">
